Commit message: Update base link dimensions and wheel separation

File: autonomous_rover/john.urdf (robot description, URDF)
Before this commit: robot john, 8 links, 7 joints
Links:
- link base_link: geometry collision box size=0.2775 0.20 0.06; visual box size=0.2775 0.20 0.06

Commit message: Adjust lidar_joint origin coordinates

File: autonomous_rover/john.urdf (robot description, URDF)
Before this commit: robot john, 8 links, 7 joints
Joints:
- joint lidar_joint: origin xyz=0.10 0.08 0.08 rpy=0 0 0 -> xyz=0.08 0.05 0.08 rpy=0 0 0

Commit message: Define inertial properties for base_footprint link
Added inertial properties to the base_footprint link.

File: autonomous_rover/john.urdf (robot description, URDF)
Before this commit: robot john, 8 links, 7 joints
Links:
- link base_footprint: mass None -> 0.0001
Joints:
- removed joint base_footprint_joint

Commit message: Add joints for base footprint and IMU link

File: autonomous_rover/john.urdf (robot description, URDF)
Before this commit: robot john, 8 links, 6 joints
Joints:
- added joint base_footprint_joint: type fixed, parent base_footprint, child base_link, origin xyz=0 0 0.06 rpy=0 0 0

Commit message: Renamed lidar_link to laser

File: autonomous_rover/john.urdf (robot description, URDF)
Before this commit: robot john, 8 links, 7 joints
Links:
- removed link lidar_link
- added link laser, mass 0.1; collision cylinder length=0.04 radius=0.035; visual cylinder length=0.04 radius=0.035
Joints:
- joint lidar_joint: child lidar_link -> laser

File: urdf/john.urdf (robot description, URDF)
Before this commit: robot john, 8 links, 7 joints
Links:
- removed link lidar_link
- added link laser, mass 0.1; collision cylinder length=0.04 radius=0.035; visual cylinder length=0.04 radius=0.035
Joints:
- joint lidar_joint: child lidar_link -> laser

Commit message: Flip base_link 180 degrees in URDF

File: autonomous_rover/john.urdf (robot description, URDF)
Before this commit: robot john, 8 links, 7 joints
Joints:
- joint base_footprint_joint: origin xyz=0 0 0.06 rpy=0 0 0 -> xyz=0 0 0.06 rpy=0 0 3.14159

File: urdf/john.urdf (robot description, URDF)
Before this commit: robot john, 8 links, 7 joints
Joints:
- joint base_footprint_joint: origin xyz=0 0 0.06 rpy=0 0 0 -> xyz=0 0 0.06 rpy=0 0 3.14159
